File: LannooLeaf.kicad_pcb (KiCad board)
At the start: 2 copper layers, 348.4 x 351.9 mm, 173 parts, among them J1 Conn_01x01, J12 Conn_02x04_Counter_Clockwise, J2 Conn_01x01, J3 Conn_01x01, J4 Conn_01x01, J5 Conn_02x04_Counter_Clockwise, J6 Conn_02x10_Counter_Clockwise, J7 Conn_02x10_Counter_Clockwise

Commit message: moved C
fixes #1
Parts:
- moved C77 12.6 mm to (240.2, 201.0)
Routing:
- net +5V: track 471.9 -> 470.1 mm
Changed lines of the file:
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@@
   )
   (footprint "Capacitor_SMD:C_0603_1608Metric" (layer "F.Cu")
-    (at 243 188.75)
+    (at 240.25 201)
     (descr "Capacitor SMD 0603 (1608 Metric), square (rectangular) end terminal, IPC_7351 nominal, (Body size source: IPC-SM-782 page 76, https://www.pcb-3d.com/wordpress/wp-content/uploads/ipc-sm-782a_amendment_1_and_2.pdf), generated with kicad-footprint-generator")
     (tags "capacitor")
@@
   (segment (start 150.43 125) (end 150.43 123.345) (width 0.5) (layer "F.Cu") (net 4))
   (segment (start 164.775 181.5) (end 164.775 181.155) (width 0.5) (layer "F.Cu") (net 4))
-  (segment (start 242.225 188.75) (end 240.5 188.75) (width 0.5) (layer "F.Cu") (net 4))
   (segment (start 95.275 190) (end 95.275 189.405) (width 0.5) (layer "F.Cu") (net 4))
   (segment (start 96.25 77.525) (end 96.275 77.5) (width 0.5) (layer "F.Cu") (net 4))
